File: Anemometer_Schematic_-_Analog_Only.sch (KiCad schematic (older format))
At the start: 44 parts, among them J1 Conn_01x10_Male, Q1 BC857, Q2 BC857, U1 LM324, U2 MAX232

Commit message: PCB draft 2
Redesigned the PCB to make the layout more optimal. Added VCC and GND connections to U1 in schematic and PCB.
Connections:
- net GND: now also U1.11 (V-), U1.11 (V-), U1.11 (V-), U1.11 (V-)
- net VCC: now also U1.4 (V+), U1.4 (V+), U1.4 (V+), U1.4 (V+)
- no-connect marks 12 -> 4
Changed lines of the file:
@@
 	1    0    0    -1
 $EndComp
-NoConn ~ 7100 2200
-NoConn ~ 7100 2800
 $Comp
 L R R17
@@
 	0    1    1    0
 $EndComp
-NoConn ~ 6050 1200
-NoConn ~ 6050 1800
 $Comp
 L R R13
@@
 	0    1    1    0
 $EndComp
-NoConn ~ 4200 1150
-NoConn ~ 4200 1750
 $Comp
 L R R10
@@
 	1    0    0    1
 $EndComp
-NoConn ~ 2300 1050
-NoConn ~ 2300 1650
 $Comp
 L R R4
@@
 	1    0    0    -1
 $EndComp
+$Comp
+L VCC #PWR020
+U 1 1 5A498E97
+P 2300 1650
+F 0 "#PWR020" H 2300 1500 50  0001 C CNN
+F 1 "VCC" H 2300 1800 50  0000 C CNN
+F 2 "" H 2300 1650 50  0001 C CNN
+F 3 "" H 2300 1650 50  0001 C CNN
+	1    2300 1650
+	1    0    0    1
+$EndComp
+$Comp
+L VCC #PWR021
+U 1 1 5A498F38
+P 4200 1750
+F 0 "#PWR021" H 4200 1600 50  0001 C CNN
+F 1 "VCC" H 4200 1900 50  0000 C CNN
+F 2 "" H 4200 1750 50  0001 C CNN
+F 3 "" H 4200 1750 50  0001 C CNN
+	1    4200 1750
+	1    0    0    1
+$EndComp
+$Comp
+L VCC #PWR022
+U 1 1 5A498FD9
+P 6050 1800
+F 0 "#PWR022" H 6050 1650 50  0001 C CNN
+F 1 "VCC" H 6050 1950 50  0000 C CNN
+F 2 "" H 6050 1800 50  0001 C CNN
+F 3 "" H 6050 1800 50  0001 C CNN
+	1    6050 1800
+	1    0    0    1
+$EndComp
+$Comp
+L VCC #PWR023
+U 1 1 5A4995FC
+P 7100 2800
+F 0 "#PWR023" H 7100 2650 50  0001 C CNN
+F 1 "VCC" H 7100 2950 50  0000 C CNN
+F 2 "" H 7100 2800 50  0001 C CNN
+F 3 "" H 7100 2800 50  0001 C CNN
+	1    7100 2800
+	1    0    0    1
+$EndComp
+$Comp
+L GND #PWR024
+U 1 1 5A499BF8
+P 7100 2200
+F 0 "#PWR024" H 7100 1950 50  0001 C CNN
+F 1 "GND" H 7100 2050 50  0000 C CNN
+F 2 "" H 7100 2200 50  0001 C CNN
+F 3 "" H 7100 2200 50  0001 C CNN
+	1    7100 2200
+	1    0    0    1
+$EndComp
+$Comp
+L GND #PWR025
+U 1 1 5A499C99
+P 6050 1200
+F 0 "#PWR025" H 6050 950 50  0001 C CNN
+F 1 "GND" H 6050 1050 50  0000 C CNN
+F 2 "" H 6050 1200 50  0001 C CNN
+F 3 "" H 6050 1200 50  0001 C CNN
+	1    6050 1200
+	1    0    0    1
+$EndComp
+$Comp
+L GND #PWR026
+U 1 1 5A49A059
+P 4200 1150
+F 0 "#PWR026" H 4200 900 50  0001 C CNN
+F 1 "GND" H 4200 1000 50  0000 C CNN
+F 2 "" H 4200 1150 50  0001 C CNN
+F 3 "" H 4200 1150 50  0001 C CNN
+	1    4200 1150
+	1    0    0    1
+$EndComp
+$Comp
+L GND #PWR027
+U 1 1 5A49A0FA
+P 2300 1050
+F 0 "#PWR027" H 2300 800 50  0001 C CNN
+F 1 "GND" H 2300 900 50  0000 C CNN
+F 2 "" H 2300 1050 50  0001 C CNN
+F 3 "" H 2300 1050 50  0001 C CNN
+	1    2300 1050
+	1    0    0    1
+$EndComp
 $EndSCHEMATC
